File: LED_Driver.sch (KiCad schematic (older format))
At the start: 0 parts

Commit message: LED Driver Module
Parts:
- added C? (x2): C, ~, symbol C
- added D?: DIODE, ~, symbol DIODE
- added L?: INDUCTOR, ~, symbol INDUCTOR
- added R?: R, ~, symbol R
- added U?: AP5726, symbol AP5726
Connections:
- net labels added: +5V, GND, LED_EN_PWM
- net labels removed: EN, FREQ
- wire segments 0 -> 20
Changed lines of the file:
@@
 Comment4 ""
 $EndDescr
-Text HLabel 2000 2750 0    60   Input ~ 0
-EN
-Text HLabel 2000 3000 0    60   Input ~ 0
-FREQ
-Text HLabel 8500 3000 0    60   Output ~ 0
+Text HLabel 3750 3000 0    60   Input ~ 0
+LED_EN_PWM
+Text HLabel 9700 1500 2    60   Output ~ 0
 String+
-Text HLabel 8500 3400 0    60   Input ~ 0
+Text HLabel 9700 2750 2    60   Input ~ 0
 String-
+$Comp
+L AP5726 U?
+U 1 1 537E69EF
+P 5250 3600
+F 0 "U?" H 4800 4850 60  0000 C CNN
+F 1 "AP5726" H 4900 4250 60  0000 C CNN
+F 2 "" H 5250 3600 60  0000 C CNN
+F 3 "" H 5250 3600 60  0000 C CNN
+	1    5250 3600
+	1    0    0    -1
+$EndComp
+$Comp
+L +5V #PWR?
+U 1 1 537E7681
+P 4100 1400
+F 0 "#PWR?" H 4100 1490 20  0001 C CNN
+F 1 "+5V" H 4100 1490 30  0000 C CNN
+F 2 "" H 4100 1400 60  0000 C CNN
+F 3 "" H 4100 1400 60  0000 C CNN
+	1    4100 1400
+	1    0    0    -1
+$EndComp
+$Comp
+L GND #PWR?
+U 1 1 537E7690
+P 4100 2400
+F 0 "#PWR?" H 4100 2400 30  0001 C CNN
+F 1 "GND" H 4100 2330 30  0001 C CNN
+F 2 "" H 4100 2400 60  0000 C CNN
+F 3 "" H 4100 2400 60  0000 C CNN
+	1    4100 2400
+	1    0    0    -1
+$EndComp
+$Comp
+L C C?
+U 1 1 537E769F
+P 4100 1950
+F 0 "C?" H 4100 2050 40  0000 L CNN
+F 1 "C" H 4106 1865 40  0000 L CNN
+F 2 "~" H 4138 1800 30  0000 C CNN
+F 3 "~" H 4100 1950 60  0000 C CNN
+	1    4100 1950
+	1    0    0    -1
+$EndComp
+$Comp
+L INDUCTOR L?
+U 1 1 537E78E3
+P 5250 1500
+F 0 "L?" V 5200 1500 40  0000 C CNN
+F 1 "INDUCTOR" V 5350 1500 40  0000 C CNN
+F 2 "~" H 5250 1500 60  0000 C CNN
+F 3 "~" H 5250 1500 60  0000 C CNN
+	1    5250 1500
+	0    -1   -1   0
+$EndComp
+$Comp
+L DIODE D?
+U 1 1 537E7B1B
+P 6350 1500
+F 0 "D?" H 6350 1600 40  0000 C CNN
+F 1 "DIODE" H 6350 1400 40  0000 C CNN
+F 2 "~" H 6350 1500 60  0000 C CNN
+F 3 "~" H 6350 1500 60  0000 C CNN
+	1    6350 1500
+	1    0    0    -1
+$EndComp
+$Comp
+L C C?
+U 1 1 537E7B28
+P 8300 2000
+F 0 "C?" H 8300 2100 40  0000 L CNN
+F 1 "C" H 8306 1915 40  0000 L CNN
+F 2 "~" H 8338 1850 30  0000 C CNN
+F 3 "~" H 8300 2000 60  0000 C CNN
+	1    8300 2000
+	1    0    0    -1
+$EndComp
+$Comp
+L GND #PWR?
+U 1 1 537E7F8D
+P 8300 2400
+F 0 "#PWR?" H 8300 2400 30  0001 C CNN
+F 1 "GND" H 8300 2330 30  0001 C CNN
+F 2 "" H 8300 2400 60  0000 C CNN
+F 3 "" H 8300 2400 60  0000 C CNN
+	1    8300 2400
+	1    0    0    -1
+$EndComp
+$Comp
+L R R?
+U 1 1 537E83D2
+P 6800 3500
+F 0 "R?" V 6880 3500 40  0000 C CNN
+F 1 "R" V 6807 3501 40  0000 C CNN
+F 2 "~" V 6730 3500 30  0000 C CNN
+F 3 "~" H 6800 3500 30  0000 C CNN
+	1    6800 3500
+	-1   0    0    1
+$EndComp
+$Comp
+L GND #PWR?
+U 1 1 537E8615
+P 4850 4050
+F 0 "#PWR?" H 4850 4050 30  0001 C CNN
+F 1 "GND" H 4850 3980 30  0001 C CNN
+F 2 "" H 4850 4050 60  0000 C CNN
+F 3 "" H 4850 4050 60  0000 C CNN
+	1    4850 4050
+	1    0    0    -1
+$EndComp
+Wire Wire Line
+	3750 3000 4250 3000
+Wire Wire Line
+	4100 1400 4100 1800
+Wire Wire Line
+	4100 2150 4100 2400
+Wire Wire Line
+	4100 1500 4950 1500
+Wire Wire Line
+	4700 1500 4700 2400
+Connection ~ 4100 1500
+Connection ~ 4700 1500
+Wire Wire Line
+	5550 1500 6150 1500
+Wire Wire Line
+	5750 1500 5750 1900
+Wire Wire Line
+	5750 1900 4950 1900
+Wire Wire Line
+	4950 1900 4950 2400
+Connection ~ 5750 1500
+Wire Wire Line
+	6550 1500 9700 1500
+Wire Wire Line
+	8300 1500 8300 1800
+Wire Wire Line
+	8300 2200 8300 2400
+Wire Wire Line
+	5450 3250 8400 3250
+Wire Wire Line
+	4850 3750 4850 4050
+Wire Wire Line
+	6800 3750 6800 3900
+Wire Wire Line
+	6800 3900 4850 3900
+Connection ~ 4850 3900
+Wire Wire Line
+	5450 3100 6800 3100
+Wire Wire Line
+	6800 3100 6800 1500
+Connection ~ 6800 1500
+Connection ~ 8300 1500
+Wire Wire Line
+	8400 3250 8400 2750
+Wire Wire Line
+	8400 2750 9700 2750
+Connection ~ 6800 3250
 $EndSCHEMATC

Commit message: Arduino Modules
Connections:
- net labels added: LED_STRING+, LED_STRING-
- net labels removed: String+, String-
Changed lines of the file:
@@
 Sheet 5 9
 Title ""
-Date "22 may 2014"
+Date "24 may 2014"
 Rev ""
 Comp ""
@@
 LED_EN_PWM
 Text HLabel 9700 1500 2    60   Output ~ 0
-String+
-Text HLabel 9700 2750 2    60   Input ~ 0
-String-
+LED_STRING+
+Text HLabel 9700 2750 2    60   Output ~ 0
+LED_STRING-
 $Comp
 L AP5726 U?
