File: Thermocouple.sch (KiCad schematic (older format))
At the start: 0 parts

Commit message: Thermocouple details
Parts:
- added C?: C, ~, symbol C
- added D?: ZENER, ~, symbol ZENER
- added R? (x7): R, ~, symbol R
- added U?: LM324, ~, symbol LM324
- added U? (x3): LM324, symbol LM324
- added U? (x2): MCP3550-60-E/SN, SO8, symbol MCP3550-60-E/SN
Connections:
- net labels added: +12V, -12V, AGND
- wire segments 0 -> 44
Other:
- note added: "16-24 bit ADC\n"
- note added: "Analog/TC Input"
- note added: "General Temperature Sensor"
- note added: "Instrumentation Amp"
